File: KiCad/nogasm/_autosave-nogasm.sch (KiCad schematic (older format))
At the start: 35 parts, among them J1 Barrel_Jack, J2 AudioJack4, J3 USB_B_Micro, Q1 AP55N03K, SW1 SW_Push, SW2 Rotary_Encoder_Switch, SW3 SW_DIP_x04, SW4 SW_DIP_x01, U1 MPXV5100DP, U2 LD29150DT50R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

Commit message: Added Autoflash for ESP32 and Center-LED
Parts:
- gave numbers to parts that had none: 1
Changed lines of the file:
@@
 	7650 5950 7750 5950
 $Comp
-L Transistor_BJT:UMH3N Q?
+L Transistor_BJT:UMH3N Q2
 U 1 1 614BD6D8
 P 6500 5350
-F 0 "Q?" H 6790 5396 50  0000 L CNN
+F 0 "Q2" H 6790 5396 50  0000 L CNN
 F 1 "UMH3N" H 6790 5305 50  0000 L CNN
 F 2 "Package_TO_SOT_SMD:SOT-363_SC-70-6" H 6505 4910 50  0001 C CNN
@@
 $EndComp
 $Comp
-L Transistor_BJT:UMH3N Q?
+L Transistor_BJT:UMH3N Q2
 U 2 1 614BFA13
 P 6500 5950
-F 0 "Q?" H 6790 5996 50  0000 L CNN
+F 0 "Q2" H 6790 5996 50  0000 L CNN
 F 1 "UMH3N" H 6790 5905 50  0000 L CNN
 F 2 "Package_TO_SOT_SMD:SOT-363_SC-70-6" H 6505 5510 50  0001 C CNN
